File: discharger/discharger.kicad_pcb (KiCad board)
At the start: 2 copper layers, 28 parts, among them J1 XT90, J2 PWR, J3 VOLT, J4 UPDI, J5 UART, Q1 2N7000, Q2 IRF4905, Q3 IRLZ44N, SW1 SW_Push, U1 LM1117-3.3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

Commit message: finish routing and gerbers
Parts:
- added SW1: PRGM/DEBUG, Button_Switch_THT:SW_Slide_1P2T_CK_OS102011MS2Q, F.Cu at (105.7, 110.0)
- added U3: L7812, Package_TO_SOT_THT:TO-220-3_Horizontal_TabDown, F.Cu at (135.6, 69.6)
- J1: footprint Connector_AMASS:AMASS_XT60-M_1x02_P7.20mm_Vertical -> discharger:XT90
- J3: footprint Connector_PinHeader_2.54mm:PinHeader_1x03_P2.54mm_Vertical -> discharger:BattMonitor
- J5: value UART -> FAN
- Q1: value 2N7000 -> 2N7002; footprint Package_TO_SOT_THT:TO-92_Inline -> Package_TO_SOT_SMD:SOT-23
- R1, R7: moved to B.Cu
- moved C1 74.0 mm to (87.9, 101.1), turned to -90 degrees
- moved R1 71.4 mm to (105.7, 104.6), turned to -90 degrees
- moved R3 68.3 mm to (104.6, 96.0), turned to 180 degrees
- moved R7 66.3 mm to (102.0, 69.6), turned to 90 degrees
- moved R5 63.9 mm to (98.0, 71.1), turned to -90 degrees
- moved R6 59.9 mm to (98.0, 78.7)
- moved R8 59.5 mm to (101.5, 66.5), turned to 180 degrees
- moved R4 59.4 mm to (94.4, 69.6)
- moved R9 58.4 mm to (102.6, 80.8), turned to -90 degrees
- moved C3 56.4 mm to (104.6, 93.5), turned to 180 degrees
- moved Q3 48.7 mm to (105.5, 78.2), turned to -90 degrees
- moved D1 47.7 mm to (91.9, 96.5)
- moved R2 41.8 mm to (109.2, 96.0), turned to 180 degrees
- moved J4 39.0 mm to (98.6, 111.8), turned to -90 degrees
- moved Q1 36.3 mm to (101.5, 71.2)
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- renumbered SW1 to START/STOP
Connections:
- J2 pad 1: Net-(C1-Pad1) -> unconnected-(J2-Pad1)
- J2 pad 2: unconnected-(J2-Pad2) -> Net-(C1-Pad1)
- J3 pad 1: +BATT -> GND
- J3 pad 3: GND -> +BATT
- J4 pad 1: /UPDI -> Net-(J4-Pad1)
- J5 pad 1: /TX -> unconnected-(J5-Pad1)
- J5 pad 2: unconnected-(J5-Pad2) -> +12V
- J5 pad 3: GND -> Net-(D2-Pad1)
- Q1 pad 1: GND -> Net-(Q1-Pad1)
- Q1 pad 2: Net-(Q1-Pad2) -> GND
- R4 pad 2: Net-(Q1-Pad2) -> Net-(Q1-Pad1)
- R5 pad 1: Net-(Q1-Pad2) -> Net-(Q1-Pad1)
Routing:
- net +BATT: track 0.00 -> 84.9 mm, vias 0 -> 1
- net +3V3: track 0.00 -> 70.6 mm
- net Net-(D2-Pad1): track 0.00 -> 64.4 mm
- net Net-(Q2-Pad2): track 0.00 -> 51.3 mm
- net /HS: track 0.00 -> 37.5 mm, vias 0 -> 2
- net GND: track 0.00 -> 32.1 mm, vias 0 -> 6
- net /LS: track 0.00 -> 24.6 mm, vias 0 -> 2
- net +12V: track 0.00 -> 21.5 mm
- net Net-(SW2-Pad1): track 0.00 -> 16.4 mm
- net Net-(C1-Pad1): track 0.00 -> 14.7 mm
- net Net-(J4-Pad1): track 0.00 -> 13.5 mm
- net Net-(C3-Pad1): track 0.00 -> 8.53 mm
- net Net-(Q3-Pad1): track 0.00 -> 6.73 mm
- net Net-(Q2-Pad1): track 0.00 -> 6.64 mm
- net Net-(Q1-Pad3): track 0.00 -> 5.60 mm
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- added copper zone on B.Cu, net GND
- added copper zone on F.Cu, net GND
Other:
- board outline added: 77.2 x 50.3 mm
- board text added: "35V MAX"
- board text added: "4.5V-15V input"
- board text added: "Battery Discharger v2 Alan Hsu"

Commit message: correct max input voltage, STEP export
Other:
- board text added: "30V MAX"
- board text removed: "35V MAX"
Changed lines of the file:
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@@
     (effects (font (size 1 1) (thickness 0.15)))
   )
-  (gr_text "35V MAX" (at 90.932 80.772 90) (layer "F.SilkS")
+  (gr_text "30V MAX" (at 90.932 80.772 90) (layer "F.SilkS")
     (effects (font (size 2 2) (thickness 0.3)))
   )
