File: discharger/discharger.kicad_pcb (KiCad board)
At the start: 2 copper layers, 77.2 x 50.3 mm, 30 parts, among them J1 XT90, J2 PWR, J3 VOLT, J4 UPDI, J5 FAN, Q1 2N7002, Q2 IRF4905, Q3 IRLZ44N, SW1 PRGM/DEBUG, U1 LM1117-3.3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

Commit message: 5V instead of 3.3V
Parts:
- U1: value LM1117-3.3 -> LM1117-5.0
- renumbered START/STOP to SW2
Connections:
- net +3V3 renamed +5V
Other:
- board text added: "6.2V-15V input"
- board text removed: "4.5V-15V input"
